Commit message: add color to my_robot & fixed *package name* in CMakeList

File: Project2/catkin_ws/src/my_robot/urdf/my_robot.xacro (robot description, xacro)
@@ -57,4 +57,5 @@
       <geometry>
         <box size=".4 .2 .1"/>
+        <material name="red"/>
       </geometry>
     </visual>
@@ -69,4 +70,5 @@
       <geometry>
         <sphere radius="0.05"/>
+        <material name="black"/>
       </geometry>
     </visual>
@@ -81,7 +83,11 @@
       <geometry>
         <sphere radius="0.05"/>
+        <material name="black"/>
       </geometry>
     </visual>
   </link>
+  <gazebo reference="chassis">
+    <material>Gazebo/Red</material>
+  </gazebo>
   <link name='left_wheel'>
     <inertial>
@@ -104,4 +110,5 @@
       <geometry>
         <cylinder radius="0.1" length="0.05"/>
+        <material name="blue"/>
       </geometry>
     </visual>
@@ -127,7 +134,14 @@
       <geometry>
         <cylinder radius="0.1" length="0.05"/>
+        <material name="blue"/>
       </geometry>
     </visual>
   </link>
+  <gazebo reference="left_wheel">
+    <material>Gazebo/Blue</material>
+  </gazebo>
+  <gazebo reference="right_wheel">
+    <material>Gazebo/Blue</material>
+  </gazebo>
   <link name='camera'>
     <pose>0 0 0 0 0 0</pose>
